File: Project/Sample-Synth/RAM_System.sch (KiCad schematic (older format))
At the start: 0 parts

Commit message: Updates and Datasheets
Included datasheets for parts chosen (so far!). Updated main schematic, separated input jacks to separate page.
Parts:
- added U?: 4017, symbol 4xxx:4017
Changed lines of the file:
@@
 $Descr A4 11693 8268
 encoding utf-8
-Sheet 3 8
+Sheet 2 8
 Title ""
 Date ""
@@
 Comment4 ""
 $EndDescr
+$Comp
+L 4xxx:4017 U?
+U 1 1 60AE7B96
+P 4100 3500
+F 0 "U?" H 4100 4481 50  0000 C CNN
+F 1 "4017" H 4100 4390 50  0000 C CNN
+F 2 "" H 4100 3500 50  0001 C CNN
+F 3 "http://www.intersil.com/content/dam/Intersil/documents/cd40/cd4017bms-22bms.pdf" H 4100 3500 50  0001 C CNN
+	1    4100 3500
+	1    0    0    -1
+$EndComp
 $EndSCHEMATC
