File: Project/Sample-Synth/DAC.sch (KiCad schematic (older format))
At the start: 0 parts

Commit message: Updates to Schematic
Schematic updates: fixed connections on RAM, started setup for DAC stage.
Also swapped out the datasheet for the RAM to a more accurate one.
Parts:
- added U? (x3): LM2904, symbol Amplifier_Operational:LM2904
Connections:
- net labels added: D0, D1, D2, D3, D4, D5, D6, D7, DACData
- wire segments 0 -> 8
Other:
- note added: "8 Bit DAC\nGoes here!"
Changed lines of the file:
@@
 $Descr A4 11693 8268
 encoding utf-8
-Sheet 1 8
+Sheet 3 8
 Title ""
 Date ""
@@
 Comment4 ""
 $EndDescr
+$Comp
+L Amplifier_Operational:LM2904 U?
+U 1 1 60B57B67
+P 4100 3550
+F 0 "U?" H 4100 3917 50  0000 C CNN
+F 1 "LM2904" H 4100 3826 50  0000 C CNN
+F 2 "" H 4100 3550 50  0001 C CNN
+F 3 "http://www.ti.com/lit/ds/symlink/lm358.pdf" H 4100 3550 50  0001 C CNN
+	1    4100 3550
+	1    0    0    -1
+$EndComp
+$Comp
+L Amplifier_Operational:LM2904 U?
+U 2 1 60B5A4FF
+P 5350 3650
+F 0 "U?" H 5350 4017 50  0000 C CNN
+F 1 "LM2904" H 5350 3926 50  0000 C CNN
+F 2 "" H 5350 3650 50  0001 C CNN
+F 3 "http://www.ti.com/lit/ds/symlink/lm358.pdf" H 5350 3650 50  0001 C CNN
+	2    5350 3650
+	1    0    0    -1
+$EndComp
+$Comp
+L Amplifier_Operational:LM2904 U?
+U 3 1 60B5C640
+P 4200 5100
+F 0 "U?" H 4158 5146 50  0000 L CNN
+F 1 "LM2904" H 4158 5055 50  0000 L CNN
+F 2 "" H 4200 5100 50  0001 C CNN
+F 3 "http://www.ti.com/lit/ds/symlink/lm358.pdf" H 4200 5100 50  0001 C CNN
+	3    4200 5100
+	1    0    0    -1
+$EndComp
+Text HLabel 1250 2900 0    50   Input ~ 0
+DACData
+Wire Bus Line
+	1250 2900 1300 2900
+Entry Wire Line
+	1300 2900 1400 3000
+Entry Wire Line
+	1300 3000 1400 3100
+Entry Wire Line
+	1300 3100 1400 3200
+Entry Wire Line
+	1300 3200 1400 3300
+Entry Wire Line
+	1300 3300 1400 3400
+Entry Wire Line
+	1300 3400 1400 3500
+Entry Wire Line
+	1300 3500 1400 3600
+Entry Wire Line
+	1300 3600 1400 3700
+Wire Wire Line
+	1400 3000 1500 3000
+Wire Wire Line
+	1400 3100 1500 3100
+Wire Wire Line
+	1400 3200 1500 3200
+Wire Wire Line
+	1400 3300 1500 3300
+Wire Wire Line
+	1400 3400 1500 3400
+Wire Wire Line
+	1400 3500 1500 3500
+Wire Wire Line
+	1400 3600 1500 3600
+Wire Wire Line
+	1400 3700 1500 3700
+Wire Bus Line
+	1300 2900 1300 3600
+Text Label 1400 3000 0    50   ~ 0
+D0
+Text Label 1400 3100 0    50   ~ 0
+D1
+Text Label 1400 3200 0    50   ~ 0
+D2
+Text Label 1400 3300 0    50   ~ 0
+D3
+Text Label 1400 3400 0    50   ~ 0
+D4
+Text Label 1400 3500 0    50   ~ 0
+D5
+Text Label 1400 3600 0    50   ~ 0
+D6
+Text Label 1400 3700 0    50   ~ 0
+D7
+Text Notes 1600 3400 0    50   ~ 0
+8 Bit DAC\nGoes here!
 $EndSCHEMATC
