File: Project/Sample-Synth/VariableClock.sch (KiCad schematic (older format))
At the start: 24 parts, among them U1 LM2904, U2 74LS628

Commit message: Updates and Datasheets
Included datasheets for parts chosen (so far!). Updated main schematic, separated input jacks to separate page.
Other:
- note added: "U1 = MCP6007\n or LM2904"
Changed lines of the file:
@@
 Wire Wire Line
 	3150 3950 3350 3950
+Text Notes 4650 3600 0    50   ~ 0
+U1 = MCP6007\n or LM2904
 $EndSCHEMATC

Commit message: Updates to Schematic
Schematic updates: fixed connections on RAM, started setup for DAC stage.
Also swapped out the datasheet for the RAM to a more accurate one.
Parts:
- RV3: value R_POT_100k -> 100k
- renumbered R4 to R5
Connections:
- net DV5 renamed D3V3
Other:
- note added: "Low pass filter stage"
- note added: "Shift and Scale"
- note added: "Sum and LPF"
- note added: "Variable oscillator input above\nOscillator output below"
- moved on the sheet: C1, C2, C3, C4, C5, C6, C7, C8, D1, R10, R11, R12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
